File: wirelss/wirelss.kicad_sch (KiCad schematic)
At the start: 10 parts

Commit message: Add files via upload
Parts:
- added C1, C2: 100uF, Capacitor_THT:CP_Axial_L10.0mm_D4.5mm_P15.00mm_Horizontal, symbol Device:C_Polarized
- D1, D2, D3: renamed from D?; footprint (none) -> LED_THT:LED_D3.0mm
- R1, R2, R3, R4, R5: renamed from R?; footprint (none) -> Resistor_THT:R_Axial_DIN0309_L9.0mm_D3.2mm_P5.08mm_Vertical
- gave numbers to parts that had none: 2
Connections:
- net GND: now also C1.2, C2.2
- net at D2.1 (K), R4.1, U2.2 (TR)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: now also C2.1
- net at R1.1, U1.2 (TR), U1.6 (THR): now also C1.1
